Commit message: fix urdf

File: drone-data/airobot.urdf (robot description, URDF)
Before this commit: robot airobot, 5 links, 4 joints
Links:
- removed link arm A
- removed link arm B
- removed link hand A
- removed link hand B
- added link armA
- added link armB
Joints:
- removed joint jointArmHandA
- removed joint jointArmHandB
- joint jointBodyArmA: child arm A -> armA
- joint jointBodyArmB: child arm B -> armB

Commit message: create world

File: drone-data/airobot.urdf (robot description, URDF)
Before this commit: robot airobot, 3 links, 2 joints
Links:
- link drone: geometry visual mesh filename=drone.dae

Commit message: Update urdf

File: drone-data/airobot.urdf (robot description, URDF)
Before this commit: robot airobot, 3 links, 2 joints
Links:
- link armA: mass None -> 0.25; geometry visual mesh filename=airobot_grip/armA.obj
- link armB: mass None -> 0.25; geometry visual mesh filename=airobot_grip/armB.obj
- link drone: mass None -> 1; geometry collision mesh filename=drone.dae; visual mesh filename=drone.dae

Commit message: fix drone model

File: drone-data/airobot.urdf (robot description, URDF)
Before this commit: robot airobot, 3 links, 2 joints
Links:
- link drone: geometry collision mesh filename=airobot.dae; visual mesh filename=airobot.dae

Commit message: fix models

File: drone-data/airobot.urdf (robot description, URDF)
Before this commit: robot airobot, 3 links, 2 joints
Joints:
- joint jointBodyArmA: origin xyz=0 -0.34 -0.44 rpy=0 0 0 -> xyz=0 0.005 0.011 rpy=0 0 0
- joint jointBodyArmB: origin xyz=0 0.34 -0.49 rpy=0 0 0 -> xyz=0 0.005 -0.011 rpy=0 0 0

Commit message: Change xyz urdf

File: drone-data/airobot.urdf (robot description, URDF)
Before this commit: robot airobot, 3 links, 2 joints
Joints:
- joint jointBodyArmA: origin xyz=0 -0.34 -0.44 rpy=0 0 0 -> xyz=-0.000648 -0.000166 0.084487 rpy=-1.5708 1.2326E-32 -2.9122E-16
- joint jointBodyArmB: origin xyz=0 0.34 -0.49 rpy=0 0 0 -> xyz=-0.000648 -0.000166 0.084487 rpy=0 0 0

Commit message: Another urdf update

File: drone-data/airobot.urdf (robot description, URDF)
Before this commit: robot airobot, 3 links, 2 joints
Links:
- link drone: geometry collision mesh filename=airobot_grip/drone.obj; visual mesh filename=airobot_grip/drone.obj

Commit message: Once again I am updating the urdf

File: drone-data/airobot.urdf (robot description, URDF)
Before this commit: robot airobot, 3 links, 2 joints
Links:
- added link world
Joints:
- added joint Fix_world: type fixed, parent world, child drone

Commit message: fix urdf

File: drone-data/airobot.urdf (robot description, URDF)
Before this commit: robot airobot, 4 links, 3 joints
Links:
- removed link world
Joints:
- removed joint Fix_world

Commit message: Add drone gripper

File: drone-data/airobot.urdf (robot description, URDF)
Before this commit: robot airobot, 3 links, 2 joints
Links:
- removed link armA
- removed link armB
Joints:
- removed joint jointBodyArmA
- removed joint jointBodyArmB
